File: single_ls403_decoder_board/schema.sch (EAGLE design)
At the start: 40 parts, among them CON1 LS403_INPUT_CONNECTOR, CON2 CONNECTOR_10PINGENERIC2X5

Commit message: New version of TTL converter ready for batch.
Parts:
- C4: value (none) -> 22uF
- CON2: PIN7 ENC_QA -> QA; PIN8 ENC_QB -> QB; PIN9 ENC_QIDX -> QIDX
Changed lines of the file:
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@@
 <part name="GND12" library="library" deviceset="GND" device=""/>
 <part name="GND6" library="library" deviceset="GND" device=""/>
-<part name="C4" library="library" deviceset="C_POL" device=""/>
+<part name="C4" library="library" deviceset="C_POL" device="" value="22uF"/>
 <part name="CON2" library="connectors" deviceset="CONNECTOR_10PIN" device="GENERIC2X5">
 <attribute name="PIN10" value="GND"/>
-<attribute name="PIN7" value="ENC_QA"/>
-<attribute name="PIN8" value="ENC_QB"/>
-<attribute name="PIN9" value="ENC_QIDX"/>
+<attribute name="PIN7" value="QA"/>
+<attribute name="PIN8" value="QB"/>
+<attribute name="PIN9" value="QIDX"/>
 </part>
 </parts>
@@
 <pinref part="R19" gate="G$1" pin="P$1"/>
 <pinref part="LM358N_2" gate="_G1" pin="-"/>
+<junction x="30.48" y="-111.76"/>
 </segment>
 </net>
@@
 <pinref part="LM393N_2" gate="_G1" pin="-"/>
 <pinref part="LM358N_2" gate="_G1" pin="OUT"/>
+<junction x="58.42" y="-114.3"/>
 </segment>
 </net>
@@
 <pinref part="R25" gate="G$1" pin="P$2"/>
 <pinref part="LM358N_2" gate="_G1" pin="+"/>
-</segment>
-</net>
+<junction x="30.48" y="-116.84"/>
+</segment>
+</net>
